Commit message: first commit

File: src/velodyne_simulator/velodyne_description/urdf/HDL-32E.urdf.xacro (robot description, xacro)
@@ -24,5 +24,5 @@
         <origin rpy="0 0 0" xyz="0 0 0.07212"/>
         <geometry>
-          <cylinder radius="0.04267" length="0.14424"/>
+          <mesh filename="package://velodyne_description/meshes/HDL32E_base.dae" />
         </geometry>
       </collision>

File: src/velodyne_simulator/velodyne_description/urdf/VLP-16.urdf.xacro (robot description, xacro)
@@ -29,5 +29,5 @@
         <origin rpy="0 0 0" xyz="0 0 0.03585"/>
         <geometry>
-          <cylinder radius="0.0516" length="0.0717"/>
+          <mesh filename="package://velodyne_description/meshes/VLP16_base_2.dae" />
         </geometry>
       </collision>
